File: eagle/verysmall-2018-pcb/verysmall-2018-sch.brd (EAGLE design)
At the start: 60 x 60 mm, 23 parts, among them IC1 7805, U1 ESP-WROOM-32, U2 AMS1117-3.3, U3 GY-521MPU6050

Commit message: ajuste de lable
Changed lines of the file:
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@@
 <param name="TopRouterVariant" value="1"/>
 <param name="tpViaShape" value="round"/>
-<param name="PrefDir.1" value="a"/>
+<param name="PrefDir.1" value="-"/>
 <param name="PrefDir.2" value="0"/>
 <param name="PrefDir.3" value="0"/>
@@
 <param name="PrefDir.14" value="0"/>
 <param name="PrefDir.15" value="0"/>
-<param name="PrefDir.16" value="a"/>
+<param name="PrefDir.16" value="|"/>
 <param name="cfVia" value="8"/>
 <param name="cfNonPref" value="5"/>
@@
 <wire x1="23.3172" y1="74.2188" x2="39.7764" y2="74.2188" width="0.1524" layer="1"/>
 <wire x1="17.2212" y1="74.2188" x2="23.3172" y2="74.2188" width="0.1524" layer="16"/>
-<wire x1="12.8016" y1="78.6384" x2="17.2212" y2="74.2188" width="0.1524" layer="16"/>
+<wire x1="12.74" y1="78.7" x2="17.2212" y2="74.2188" width="0.1524" layer="16"/>
 <wire x1="39.7764" y1="74.2188" x2="39.87" y2="74.255" width="0.1524" layer="1"/>
-<wire x1="12.8016" y1="78.6384" x2="12.74" y2="78.7" width="0.1524" layer="16"/>
 <via x="23.3172" y="74.2188" extent="1-16" drill="0.35"/>
 </signal>
