File: eagle/verysmall-2018-pcb/verysmall-2018-sch.brd (EAGLE design)
At the start: 65 x 66 mm, 37 parts, among them IC1 7805, Q1 BC548, U1 ESP-WROOM-32, U2 AMS1117-3.3, U3 GY-521MPU6050

Commit message: atualizando
Parts:
- removed MOTOR-A, MOTOR-B: (no value), con-molex:KK-156-2
- removed R3: 1M, rcl:0204/7
- removed R5: 2K2, eagle-ltspice:0207/10
- removed R6: 2M, rcl:0204/7
- added D2: 1N540x, diode:DO201-15
- added MOTOR_A, MOTOR_B: (no value), pinhead:1X02
- added R8: 2k2, rcl:0204/7
- BAT: device con-molex:KK-156-2 -> pinhead:1X02
- D1: device 1N4007:DIOAD1060W80L520D270 -> diode:D-7.5
- R1: value 10M -> 100k
- R2: value 2.4M -> 10k
- R4: value 220 -> 150
- U$1: value MP1584 -> MP1584-MINI-SMD; device MP1584-dc-brick:DC-BRICK -> MP1584-dc-brick:MINI-DC-BRICK-SMD
- moved JP2 33.6 mm to (35.6, 37.2)
- moved C4 21.6 mm to (47.0, 53.7), turned to 270 degrees
- moved U$1 13.3 mm to (24.5, 54.6)
- moved R4 9.62 mm to (5.50, 73.4), turned to 90 degrees
- moved LED1 6.40 mm to (9.10, 84.9), turned to 90 degrees
- moved U3 3.40 mm to (12.3, 45.2)
- moved D1 3.32 mm to (33.7, 87.4), flipped to the top, turned to 180 degrees
- moved C1 3.00 mm to (41.3, 86.6), turned to 270 degrees
- moved R7 2.50 mm to (45.5, 73.0)
- moved S2 2.33 mm to (23.0, 75.5), turned to 180 degrees
- moved C8 1.88 mm to (19.3, 42.1), turned to 359.6 degrees
- moved BAT 1.46 mm to (44.2, 94.8)
- moved SV1 1.00 mm to (42.5, 56.6)
- moved Q1 0.71 mm to (3.79, 87.0)
Connections:
- net N$1 renamed SCL
- net N$3 renamed SDA
- net N$4 renamed EN
- net N$9 renamed GPIO0
- removed net N$17: Q1.C, SG2.+
- removed net N$18: Q1.B, R5.2
- removed net N$2: R2.1, R3.2
- new net N$1: C8.1, D2.C, U$1.P$2
- new net N$10: Q1.C, SG2.-
- new net N$14: Q1.B, R8.1
- net 5V: now also SG2.+; no longer SG2.-
- net A01: now also MOTOR_A.2; no longer MOTOR-A.2
- net A02: now also MOTOR_A.1; no longer MOTOR-A.1
- net AI1: now also U1.11; no longer U1.8
- net AI2: now also U1.10; no longer U1.7
- net B01: now also MOTOR_B.1; no longer MOTOR-B.1
- net B02: now also MOTOR_B.2; no longer MOTOR-B.2
- net BAT_VCC: now also D2.A; no longer C8.1, U$1.IN+1, U$1.IN+2
- net BI1: now also U1.12; no longer U1.10
- net BI2: now also U1.13; no longer U1.11
- net BUZZER: now also R8.2; no longer R5.1
- net GND: now also R2.1, U$1.P$1, U$1.P$4; no longer R3.1, U$1.IN-1, U$1.IN-2, U$1.OUT-1, U$1.OUT-2
- net N$7: no longer R6.2
- net PWMA: now also U1.8; no longer U1.6
- net PWMB: now also U1.14; no longer U1.12
- net VM: now also U$1.P$3; no longer U$1.OUT+1, U$1.OUT+2
- net V_OUT: no longer R6.1
Routing:
- net GND: track 24.1 -> 148.5 mm
- net BAT_VCC: track 90.7 -> 23.6 mm, vias 1 -> 0
- net N$1: track 0.00 -> 40.4 mm
- net N$10: track 0.00 -> 16.3 mm
- net GPIO0: track 22.1 -> 38.3 mm
- net N$17: track 13.9 -> 0.00 mm
- net LED: track 24.0 -> 12.8 mm
- net EN: track 47.7 -> 54.9 mm
- net 5V: track 112.0 -> 104.9 mm
- net N$2: track 6.64 -> 0.00 mm
- net N$18: track 5.69 -> 0.00 mm
- net SDA: track 6.57 -> 11.7 mm
- net N$14: track 0.00 -> 4.76 mm
- net B02: track 17.1 -> 21.5 mm
- net BUZZER: track 25.5 -> 29.7 mm
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