File: eagle/verysmall-2018-pcb/verysmall-2018-sch.sch (EAGLE design)
At the start: 37 parts, among them IC1 7805, Q1 BC548, U1 ESP-WROOM-32, U2 AMS1117-3.3, U3 GY-521MPU6050

Commit message: atualizando
Parts:
- removed MOTOR-A, MOTOR-B: (no value), con-molex:KK-156-2
- removed R3: 1M, rcl:R-EU_0204/7
- removed R5: 2K2, eagle-ltspice:R0207/10
- removed R6: 2M, rcl:R-EU_0204/7
- added D2: 1N540x, diode:1N5400
- added MOTOR_A, MOTOR_B: (no value), pinhead:PINHD-1X2
- added R8: 2k2, rcl:R-EU_0204/7
- BAT: device con-molex:KK-156-2 -> pinhead:PINHD-1X2
- D1: device 1N4007:1N4007 -> diode:DIODE-D-7.5
- R1: value 10M -> 100k
- R2: value 2.4M -> 10k
- R4: value 220 -> 150
- U$1: value MP1584 -> MP1584-MINI-SMD; device MP1584-dc-brick:MP1584 -> MP1584-dc-brick:MP1584-MINI-SMD
Connections:
- net N$1 renamed SCL
- net N$3 renamed SDA
- net N$4 renamed EN
- net N$9 renamed GPIO0
- removed net N$17: Q1.C, SG2.-
- removed net N$18: Q1.B, R5.2
- removed net N$2: R2.1, R3.2
- new net N$1: C8.1, D2.C, U$1.VIN+
- new net N$10: Q1.C, SG2.+
- new net N$14: Q1.B, R8.1
- net 5V: now also SG2.-; no longer SG2.+
- net A01: now also MOTOR_A.2; no longer MOTOR-A-2.S
- net A02: now also MOTOR_A.1; no longer MOTOR-A-1.S
- net AI1: now also U1.IO26; no longer U1.IO32
- net AI2: now also U1.IO25; no longer U1.IO35
- net B01: now also MOTOR_B.1; no longer MOTOR-B-1.S
- net B02: now also MOTOR_B.2; no longer MOTOR-B-2.S
- net BAT_VCC: now also D2.A; no longer C8.1, U$1.VIN+
- net BI1: now also U1.IO27; no longer U1.IO25
- net BI2: now also U1.IO14; no longer U1.IO26
- net BUZZER: now also R8.2; no longer R5.1
- net GND: now also BAT.1, R2.1; no longer BAT-1.S, R3.1
- net N$7: no longer R6.2
- net N$8: now also BAT.2; no longer BAT-2.S
- net PWMA: now also U1.IO32; no longer U1.IO34
- net PWMB: now also U1.IO12; no longer U1.IO27
- net V_OUT: no longer R6.1
Other:
- moved on the sheet: C3, D1, JP2, SG2
